File: touch_panel.kicad_sch (KiCad schematic)
At the start: 52 parts, among them J1 2x4 SMD 2.0 MM, J2 2x4 Regular, Q1 MMBT2222, Q2 MMBT2222, Q3 MMBT2222, Q4 MMBT2222, Q5 MMBT2222, Q6 MMBT2222, SW1 Reset Switch, U1 TTP223_1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

Commit message: Board finalized for printing
Parts:
- removed C1, C3, C5: 0-50 pF (30 pF), Capacitor_Tantalum_SMD:CP_EIA-1608-10_AVX-L_Pad1.25x1.05mm_HandSolder, symbol Device:C
- removed C2, C4, C6: 100nF, Capacitor_Tantalum_SMD:CP_EIA-1608-10_AVX-L_Pad1.25x1.05mm_HandSolder, symbol Device:C
- removed D1, D3, D5: BLUE, LED_SMD:LED_0603_1608Metric_Pad1.05x0.95mm_HandSolder, symbol Device:LED
- removed D2, D6: WHITE, LED_SMD:LED_0603_1608Metric_Pad1.05x0.95mm_HandSolder, symbol Device:LED
- removed D7, D8, D9: RED, LED_SMD:LED_0603_1608Metric_Pad1.05x0.95mm_HandSolder, symbol Device:LED
- removed J1: 2x4 SMD 2.0 MM, Connector_PinHeader_2.00mm:PinHeader_2x04_P2.00mm_Vertical, symbol Connector_Generic:Conn_02x04_Counter_Clockwise
- removed J2: 2x4 Regular, Connector_PinHeader_2.00mm:PinHeader_2x04_P2.00mm_Vertical, symbol Connector_Generic:Conn_02x03_Counter_Clockwise
- removed PAD1: Sense pad 1, Connector:senspad, symbol Device:Sense_pad
- removed PAD2: Sense pad 2, Connector:senspad, symbol Device:Sense_pad
- removed PAD3: Sense pad 3, Connector:senspad, symbol Device:Sense_pad
- removed Q1, Q2, Q3, Q4, Q5, Q6: MMBT2222, Package_TO_SOT_SMD:TSOT-23, symbol Transistor_BJT:2N2219
- removed R10, R14, R16, R8: 10K, Resistor_SMD:R_0603_1608Metric_Pad0.98x0.95mm_HandSolder, symbol Device:R
- removed R11, R12, R17, R18: 10R, Resistor_SMD:R_0603_1608Metric_Pad0.98x0.95mm_HandSolder, symbol Device:R
- removed R13, R15, R19, R20, R21, R9: 1K, Resistor_SMD:R_0603_1608Metric_Pad0.98x0.95mm_HandSolder, symbol Device:R
- removed SW1: Reset Switch, Button_Switch_SMD:SW_Push_1P1T_NO_6x6mm_H9.5mm, symbol Switch:SW_Push
- removed U1: TTP223_1, ttp223:SOT95P285X126-6N, symbol ttp223:TTP223_
- removed U2: TTP223_2, ttp223:SOT95P285X126-6N, symbol ttp223:TTP223_
- removed U3: TTP223_3, ttp223:SOT95P285X126-6N, symbol ttp223:TTP223_
- removed U4: ESP-12E, RF_Module:ESP-12E, symbol RF_Module:ESP-12E
- added C1, C2: 22uF, Capacitor_Tantalum_SMD:CP_EIA-1608-10_AVX-L, symbol Device:C_Polarized_Small_US
- added D1, D2, D3: DIODE, Diode_SMD:D_2114_3652Metric_Pad1.85x3.75mm_HandSolder, symbol Simulation_SPICE:DIODE
- added J1: Screw_Terminal_01x06, Converter_ACDC:touch-relay, symbol Connector:Screw_Terminal_01x06
- added J2: 2x4 SMD 2.0 MM, Connector_PinHeader_2.00mm:PinHeader_2x04_P2.00mm_Vertical, symbol Connector_Generic:Conn_02x04_Counter_Clockwise
- added PS1: HLK-PM01, Converter_ACDC:Converter_ACDC_HiLink_HLK-PMxx, symbol Converter_ACDC:HLK-PM01
- added Q1, Q2, Q3: MMBT2222*, MMBT:SOT23-BEC, symbol mmbt2222:MMBT2222*
- added U1, U2, U3: c0942, Relay_THT:c0942, symbol Relay:c0942
- added U4: AMS1117-3.3, Package_TO_SOT_SMD:SOT-223-3_TabPin2, symbol Regulator_Linear:AMS1117-3.3
- D4: value WHITE -> RED
- R5: value 10R -> 1K
- R6: value 10R -> 10K
- R7: value 1K -> 2K
Connections:
- net BLUELED is gone; now on an unnamed net: R3.1
- net +3V3: now also C2.1, J2.1 (Pin_1), U4.2 (VO); no longer D4.2 (A)
- net GND: now also D4.1 (K), R6.1, C1.2, C2.2, J2.8 (Pin_8), PS1.3 (-Vout), Q1.E, Q2.E, Q3.E, U4.1 (GND)
- net Relay 1: now also R1.2, J2.4 (Pin_4); no longer R1.1
- net Relay 2: now also R3.2, J2.3 (Pin_3); no longer R7.1
- net Relay 3: now also R5.2, J2.6 (Pin_6)
- net at R6.2: now also R5.1, Q3.B
- net +5V: now reaches R7.2
- net +5V: now also C1.1, D1.2 (K), D2.2 (K), D3.2 (K), PS1.4 (+Vout), U1.3, U2.3, U3.3, U4.3 (VI)
- net at R4.2: now also Q2.B; no longer R3.2
- net at R2.2: now also R1.1, Q1.B; no longer R1.2
- new net: D2.1 (A), Q2.C, U2.4
- new net: D3.1 (A), Q3.C, U3.4
- new net: D1.1 (A), Q1.C, U1.4
- new net: D4.2 (A), R7.1
- new net Load 1: J1.4 (Pin_4), U1.1, U1.14
- new net Load 2: J1.5 (Pin_5), U2.1, U2.14
- new net Load 3: J1.6 (Pin_6), U3.1, U3.14
- new net Neutral: J1.2 (Pin_2), PS1.1 (AC/L)
- new net Phase: J1.1 (Pin_1), PS1.2 (AC/N), U1.2, U1.8, U2.2, U2.8, U3.2, U3.8
- no-connect marks 13 -> 4
Other:
- note removed: "ESP-12"
- note removed: "LED Indicators 1"
- note removed: "LED Indicators 2"
- note removed: "LED Indicators 3"
- note removed: "Touch sensors 1"
- note removed: "Touch sensors 2"
- note removed: "Touch sensors 3"
